File: FlatSat-A/FlatSat-A.kicad_sch (KiCad schematic)
At the start: 21 parts, among them J1 LiPo, U2 MPU-6050, U3 BME280

Commit message: add inital PCB design
Parts:
- removed R1, R2, R3, R6, R7: 10K, symbol Device:R_Small_US
- added J4, J5: Conn_01x04_MountingPin, symbol Connector_Generic_MountingPin:Conn_01x04_MountingPin
- added JP2, JP3, JP5: SolderJumper_2_Bridged, Jumper:SolderJumper-2_P1.3mm_Bridged_RoundedPad1.0x1.5mm, symbol Jumper:SolderJumper_2_Bridged
- added RN1: 10K, symbol Device:R_Pack04_Split
- added TP1, TP2: TestPoint, symbol Connector:TestPoint
- JP1: footprint (none) -> Jumper:SolderJumper-2_P1.3mm_Bridged_RoundedPad1.0x1.5mm
- U1: value ~ -> Xiao; footprint (none) -> LyndLabs Footprints:XIAO-Generic
- U4: value ~ -> MiniMeter
Connections:
- net +3V3: now also U5.8 (VCC), U6.8 (VCC), J4.2 (Pin_2), J5.2 (Pin_2), RN1.5 (R4.2), RN1.6 (R3.2), RN1.7 (R2.2), RN1.8 (R1.2); no longer U5.1 (VCC), U6.1 (VCC)
- net CS1: now also U5.6 (NSS); no longer U5.3 (NSS)
- net CS2: now also U6.6 (NSS); no longer U6.3 (NSS)
- net GND: now also U5.7 (GND), U6.7 (GND), J4.1 (Pin_1), J4.MP (MountPin), J5.1 (Pin_1), J5.MP (MountPin); no longer U5.2 (GND), U6.2 (GND)
- net MISO: now also U5.2 (MISO), U6.2 (MISO); no longer U5.7 (MISO), U6.7 (MISO)
- net MOSI: now also U5.3 (MOSI), U6.3 (MOSI); no longer U5.6 (MOSI), U6.6 (MOSI)
- net SCK: now also U5.4 (CLK), U6.4 (CLK); no longer U5.5 (CLK), U6.5 (CLK)
- net SCL: now also J5.4 (Pin_4), RN1.2 (R2.1)
- net SDA: now also J5.3 (Pin_3), RN1.1 (R1.1)
- net INT: now reaches U1.4 (D3)
- net INT: now also JP2.2 (B)
- net MCU_TX: now reaches U1.7 (TX)
- net MCU_TX: now also J4.4 (Pin_4)
- net MCU_RX: now reaches U1.8 (RX)
- net MCU_RX: now also J4.3 (Pin_3)
- net at U5.11 (BUSY): now also JP3.1 (A)
- net at U5.12 (DI01): now also TP1.1
- net at U2.12 (INT): now also JP2.1 (A)
- net at U6.11 (BUSY): now also JP5.1 (A)
- net at U6.12 (DI01): now also TP2.1
- new net: RN1.4 (R4.1), U6.5 (RST)
- new net: RN1.3 (R3.1), U5.5 (RST)
- new net BUSY1: JP3.2 (B)
- new net BUSY2: JP5.2 (B)
Other:
- note added: "Qwiic Connector"
