File: src/FlatSat.kicad_pcb (KiCad board)
At the start: 2 copper layers, 48 x 32 mm, 35 parts, among them J1 LiPo, J2 Conn_01x04_MountingPin, J3 Conn_01x04_MountingPin, J4 Conn_02x03_Odd_Even, J5 Conn_01x12_Pin, J7 Micro_SD_Card, U1 Xiao, U2 MPU-6050, U3 BME280, U4 MiniMeter

Commit message: push v0.1 - MPU6500 compat & production files
Parts:
- removed R6: 10K, Resistor_SMD:R_0603_1608Metric
- added C6: 100nF, Capacitor_SMD:C_0603_1608Metric_Pad1.08x0.95mm_HandSolder, F.Cu at (-16.7, 12.7)
- added JP4: SolderJumper_2_Open, Jumper:SolderJumper-2_P1.3mm_Open_RoundedPad1.0x1.5mm, B.Cu at (10.2, 3.76)
- added JP6: SolderJumper_2_Bridged, Jumper:SolderJumper-2_P1.3mm_Bridged_RoundedPad1.0x1.5mm, B.Cu at (10.6, 0.79)
- C3: value 0.1uf -> 100nF
- J7: value Micro_SD_Card -> Micro_SD_Card_Det2
- R4, R5: value 10K -> 4.7K
- U2: value MPU-6050 -> MPU-6050 / 6500
- U3: value BME280 -> BME280 /BMP280
- moved U3 1.34 mm to (-13.6, 13.5)
- moved C3 0.78 mm to (-16.8, 14.1), turned to 180 degrees
- moved RN1 0.75 mm to (10.0, -0.75)
Connections:
- C2 pad 1: Net-(U2-CPOUT) -> Net-(JP4-B)
- J7 pad 10: (no net) -> SD_DT
- U1 pad 22: unconnected-(U1-D18-Pad22) -> SD_DT
- U2 pad 20: Net-(U2-CPOUT) -> Net-(JP4-A)
- U2 pad 22: unconnected-(U2-RESV-Pad22) -> NCS
- U3 pad 2: Net-(U3-CSB) -> +3V3
Routing:
- net SD_DT: track 0.00 -> 27.4 mm, vias 0 -> 1
- net GND: track 6.85 -> 24.7 mm, vias 61 -> 36
- net Net-(JP4-A): track 0.00 -> 6.07 mm, vias 0 -> 1
- net SDA: track 82.4 -> 78.0 mm
- net NCS: track 0.00 -> 3.64 mm, vias 0 -> 1
- net Net-(U2-CPOUT): track 3.51 -> 0.00 mm
- net +3V3: track 173.2 -> 176.5 mm
- net Net-(JP4-B): track 0.00 -> 3.09 mm, vias 0 -> 1
- net A1: track 44.9 -> 47.6 mm
- net SCL: track 84.4 -> 82.6 mm
- net Net-(U3-CSB): track 1.46 -> 0.00 mm
- net LED: track 44.4 -> 43.0 mm
- net Net-(RN1D-R4.2): track 9.12 -> 9.96 mm
- net VCC: track 83.2 -> 82.5 mm
- net SCK: track 61.3 -> 61.9 mm
Other:
- board text added: "Learn more at pwnsat.org"
- board text added: "v0.1"
- board text removed: "Learn more at flatsat.org"
- board text removed: "v0.0"

Commit message: push FlatSat enclosure
Parts:
- U2: footprint Sensor_Motion:InvenSense_QFN-24_4x4mm_P0.5mm -> Package_DFN_QFN:QFN-24-1EP_3x3mm_P0.4mm_EP1.75x1.6mm
- moved U2 0.39 mm to (5.20, -1.00)
Routing:
- net SDA: track 78.0 -> 79.3 mm
- net +3V3: track 176.5 -> 177.7 mm
- net Net-(JP4-A): track 6.07 -> 7.08 mm
- net SCL: track 82.6 -> 83.4 mm
- net NCS: track 3.64 -> 4.48 mm
- net Net-(JP2-A): track 5.96 -> 6.63 mm
- net GND: track 24.7 -> 25.4 mm
